File: deskav2.brd (EAGLE design)
At the start: 50.5 x 68.6 mm, 23 parts, among them Q1 BC547, Q2 BC547

Commit message: v0.6 + reconnect each 10 minutes
Parts:
- removed BUZZER, LED: (no value), con-wago-508:W237-132
- added SL5, SL6: (no value), con-amp-quick:02P
- moved R4 7.67 mm to (15.9, 18.4), turned to 270 degrees
- moved R5 7.67 mm to (27.9, 18.4), turned to 270 degrees
- moved SL1 3.81 mm to (47.0, 47.6)
- moved SL2 1.27 mm to (47.0, 45.1)
- moved SL3 0.63 mm to (47.0, 42.5)
- renumbered X1 to RELAY
Connections:
- net +5V: now also SL5.2, SL6.1; no longer BUZZER.2, LED.2
- net N$15: now also SL6.2; no longer BUZZER.1
- net N$6: now also SL5.1; no longer LED.1
Routing:
- net +5V: track 192.8 -> 171.7 mm
- net N$12: track 42.1 -> 29.7 mm
- net N$11: track 29.6 -> 17.3 mm
- net GND: track 161.0 -> 149.6 mm
- net N$4: track 19.3 -> 10.2 mm
- net N$13: track 5.75 -> 13.0 mm
- net N$5: track 10.5 -> 5.71 mm
- net N$10: track 20.2 -> 23.5 mm
- net N$6: track 13.0 -> 10.1 mm
- net N$9: track 17.9 -> 15.9 mm
- net N$14: track 9.46 -> 11.2 mm
- net N$8: track 34.3 -> 33.0 mm
- net N$17: track 29.4 -> 28.4 mm
- net N$3: track 17.0 -> 17.9 mm
