File: deskav2.sch (EAGLE design)
At the start: 23 parts, among them Q1 BC547, Q2 BC547

Commit message: v0.6 + reconnect each 10 minutes
Parts:
- removed BUZZER, LED: (no value), con-wago-508:W237-02P
- added SL5, SL6: (no value), con-amp-quick:M02
- renumbered X1 to RELAY
Connections:
- net +5V: now also SL5.2, SL6.1; no longer BUZZER-2.KL, LED-2.KL
- net N$15: now also SL6.2; no longer BUZZER-1.KL
- net N$6: now also SL5.1; no longer LED-1.KL
Changed lines of the file:
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@@
 <grid distance="0.1" unitdist="inch" unit="inch" style="lines" multiple="1" display="no" altdistance="0.01" altunitdist="inch" altunit="inch"/>
 <layers>
-<layer number="1" name="Top" color="4" fill="1" visible="no" active="no"/>
-<layer number="16" name="Bottom" color="1" fill="1" visible="no" active="no"/>
-<layer number="17" name="Pads" color="2" fill="1" visible="no" active="no"/>
-<layer number="18" name="Vias" color="2" fill="1" visible="no" active="no"/>
-<layer number="19" name="Unrouted" color="6" fill="1" visible="no" active="no"/>
-<layer number="20" name="Dimension" color="15" fill="1" visible="no" active="no"/>
-<layer number="21" name="tPlace" color="7" fill="1" visible="no" active="no"/>
-<layer number="22" name="bPlace" color="7" fill="1" visible="no" active="no"/>
-<layer number="23" name="tOrigins" color="15" fill="1" visible="no" active="no"/>
-<layer number="24" name="bOrigins" color="15" fill="1" visible="no" active="no"/>
-<layer number="25" name="tNames" color="7" fill="1" visible="no" active="no"/>
-<layer number="26" name="bNames" color="7" fill="1" visible="no" active="no"/>
-<layer number="27" name="tValues" color="7" fill="1" visible="no" active="no"/>
-<layer number="28" name="bValues" color="7" fill="1" visible="no" active="no"/>
+<layer number="1" name="Top" color="4" fill="1" visible="yes" active="no"/>
+<layer number="16" name="Bottom" color="1" fill="1" visible="yes" active="no"/>
+<layer number="17" name="Pads" color="2" fill="1" visible="yes" active="no"/>
+<layer number="18" name="Vias" color="2" fill="1" visible="yes" active="no"/>
+<layer number="19" name="Unrouted" color="6" fill="1" visible="yes" active="no"/>
+<layer number="20" name="Dimension" color="15" fill="1" visible="yes" active="no"/>
+<layer number="21" name="tPlace" color="7" fill="1" visible="yes" active="no"/>
+<layer number="22" name="bPlace" color="7" fill="1" visible="yes" active="no"/>
+<layer number="23" name="tOrigins" color="15" fill="1" visible="yes" active="no"/>
+<layer number="24" name="bOrigins" color="15" fill="1" visible="yes" active="no"/>
+<layer number="25" name="tNames" color="7" fill="1" visible="yes" active="no"/>
+<layer number="26" name="bNames" color="7" fill="1" visible="yes" active="no"/>
+<layer number="27" name="tValues" color="7" fill="1" visible="yes" active="no"/>
+<layer number="28" name="bValues" color="7" fill="1" visible="yes" active="no"/>
 <layer number="29" name="tStop" color="7" fill="3" visible="no" active="no"/>
 <layer number="30" name="bStop" color="7" fill="6" visible="no" active="no"/>
@@
 <layer number="35" name="tGlue" color="7" fill="4" visible="no" active="no"/>
 <layer number="36" name="bGlue" color="7" fill="5" visible="no" active="no"/>
-<layer number="37" name="tTest" color="7" fill="1" visible="no" active="no"/>
-<layer number="38" name="bTest" color="7" fill="1" visible="no" active="no"/>
+<layer number="37" name="tTest" color="7" fill="1" visible="yes" active="no"/>
+<layer number="38" name="bTest" color="7" fill="1" visible="yes" active="no"/>
 <layer number="39" name="tKeepout" color="4" fill="11" visible="no" active="no"/>
 <layer number="40" name="bKeepout" color="1" fill="11" visible="no" active="no"/>
@@
 <layer number="44" name="Drills" color="7" fill="1" visible="no" active="no"/>
 <layer number="45" name="Holes" color="7" fill="1" visible="no" active="no"/>
-<layer number="46" name="Milling" color="3" fill="1" visible="no" active="no"/>
-<layer number="47" name="Measures" color="7" fill="1" visible="no" active="no"/>
-<layer number="48" name="Document" color="7" fill="1" visible="no" active="no"/>
-<layer number="49" name="Reference" color="7" fill="1" visible="no" active="no"/>
-<layer number="51" name="tDocu" color="7" fill="1" visible="no" active="no"/>
-<layer number="52" name="bDocu" color="7" fill="1" visible="no" active="no"/>
+<layer number="46" name="Milling" color="3" fill="1" visible="yes" active="no"/>
+<layer number="47" name="Measures" color="7" fill="1" visible="yes" active="no"/>
+<layer number="48" name="Document" color="7" fill="1" visible="yes" active="no"/>
+<layer number="49" name="Reference" color="7" fill="1" visible="yes" active="no"/>
+<layer number="51" name="tDocu" color="7" fill="1" visible="yes" active="no"/>
+<layer number="52" name="bDocu" color="7" fill="1" visible="yes" active="no"/>
 <layer number="90" name="Modules" color="5" fill="1" visible="yes" active="yes"/>
 <layer number="91" name="Nets" color="2" fill="1" visible="yes" active="yes"/>
@@
 <part name="R3" library="rcl" deviceset="R-EU_" device="0207/7" value="4k7"/>
 <part name="GND1" library="supply1" deviceset="GND" device=""/>
-<part name="LED" library="con-wago-508" deviceset="W237-02P" device=""/>
 <part name="R4" library="rcl" deviceset="R-EU_" device="0207/7" value="220"/>
-<part name="BUZZER" library="con-wago-508" deviceset="W237-02P" device=""/>
 <part name="DALLAS" library="con-wago-508" deviceset="W237-3E" device=""/>
 <part name="Q1" library="transistor-npn" deviceset="BC547*" device=""/>
@@
 <part name="GND7" library="supply1" deviceset="GND" device=""/>
 <part name="COMMUNIT1" library="con-wago-508" deviceset="W237-04P" device=""/>
-<part name="X1" library="con-wago-508" deviceset="W237-3E" device=""/>
+<part name="RELAY" library="con-wago-508" deviceset="W237-3E" device=""/>
 <part name="GND8" library="supply1" deviceset="GND" device=""/>
 <part name="SL1" library="con-amp-quick" deviceset="M04" device=""/>
@@
 <part name="P+7" library="supply1" deviceset="+5V" device=""/>
 <part name="GND9" library="supply1" deviceset="GND" device=""/>
+<part name="SL5" library="con-amp-quick" deviceset="M02" device=""/>
+<part name="SL6" library="con-amp-quick" deviceset="M02" device=""/>
 </parts>
 <sheets>
@@
 <instance part="R3" gate="G$1" x="15.24" y="68.58" rot="R90"/>
 <instance part="GND1" gate="1" x="-25.4" y="35.56"/>
-<instance part="LED" gate="-1" x="12.7" y="33.02" rot="R90"/>
-<instance part="LED" gate="-2" x="10.16" y="33.02" rot="R90"/>
 <instance part="R4" gate="G$1" x="20.32" y="38.1" rot="R180"/>
-<instance part="BUZZER" gate="-1" x="114.3" y="58.42" rot="R180"/>
-<instance part="BUZZER" gate="-2" x="114.3" y="60.96" rot="R180"/>
 <instance part="DALLAS" gate="-1" x="-7.62" y="78.74"/>
 <instance part="DALLAS" gate="-2" x="-7.62" y="76.2"/>
@@
 <instance part="COMMUNIT1" gate="-3" x="86.36" y="48.26" rot="R180"/>
 <instance part="COMMUNIT1" gate="-4" x="86.36" y="45.72" rot="R180"/>
-<instance part="X1" gate="-1" x="-33.02" y="73.66"/>
-<instance part="X1" gate="-2" x="-33.02" y="71.12"/>
-<instance part="X1" gate="-3" x="-33.02" y="68.58"/>
+<instance part="RELAY" gate="-1" x="-33.02" y="73.66"/>
+<instance part="RELAY" gate="-2" x="-33.02" y="71.12"/>
+<instance part="RELAY" gate="-3" x="-33.02" y="68.58"/>
 <instance part="GND8" gate="1" x="-27.94" y="63.5"/>
 <instance part="SL1" gate="G$1" x="88.9" y="86.36" rot="R270"/>
@@
 <instance part="P+7" gate="1" x="-20.32" y="132.08"/>
 <instance part="GND9" gate="1" x="-20.32" y="96.52"/>
+<instance part="SL5" gate="G$1" x="12.7" y="30.48" rot="R90"/>
+<instance part="SL6" gate="G$1" x="116.84" y="60.96" rot="R180"/>
 </instances>
 <busses>
@@
 </segment>
 <segment>
-<pinref part="X1" gate="-3" pin="KL"/>
+<pinref part="RELAY" gate="-3" pin="KL"/>
 <pinref part="GND8" gate="1" pin="GND"/>
 <wire x1="-27.94" y1="68.58" x2="-27.94" y2="66.04" width="0.1524" layer="91"/>
@@
 <net name="N$6" class="0">
 <segment>
-<pinref part="LED" gate="-1" pin="KL"/>
 <pinref part="R4" gate="G$1" pin="2"/>
 <wire x1="12.7" y1="38.1" x2="15.24" y2="38.1" width="0.1524" layer="91"/>
+<pinref part="SL5" gate="G$1" pin="1"/>
 </segment>
 </net>
@@
 <net name="N$15" class="0">
 <segment>
-<pinref part="BUZZER" gate="-1" pin="KL"/>
 <pinref part="Q1" gate="G$1" pin="C"/>
 <wire x1="109.22" y1="58.42" x2="109.22" y2="45.72" width="0.1524" layer="91"/>
+<pinref part="SL6" gate="G$1" pin="2"/>
 </segment>
 </net>
@@
 <net name="+5V" class="0">
 <segment>
-<pinref part="LED" gate="-2" pin="KL"/>
 <pinref part="P+3" gate="1" pin="+5V"/>
 <wire x1="10.16" y1="38.1" x2="5.08" y2="38.1" width="0.1524" layer="91"/>
+<pinref part="SL5" gate="G$1" pin="2"/>
 </segment>
 <segment>
@@
 <wire x1="91.44" y1="66.04" x2="91.44" y2="60.96" width="0.1524" layer="91"/>
 <junction x="91.44" y="66.04"/>
-<pinref part="BUZZER" gate="-2" pin="KL"/>
 <wire x1="91.44" y1="60.96" x2="109.22" y2="60.96" width="0.1524" layer="91"/>
 <pinref part="SL1" gate="G$1" pin="3"/>
@@
 <pinref part="SL3" gate="G$1" pin="3"/>
 <pinref part="SL4" gate="G$1" pin="3"/>
+<pinref part="SL6" gate="G$1" pin="1"/>
 </segment>
 <segment>
@@
 </segment>
 <segment>
-<pinref part="X1" gate="-1" pin="KL"/>
+<pinref part="RELAY" gate="-1" pin="KL"/>
 <pinref part="P+1" gate="1" pin="+5V"/>
 <wire x1="-27.94" y1="73.66" x2="-27.94" y2="76.2" width="0.1524" layer="91"/>
@@
 <net name="N$14" class="0">
 <segment>
-<pinref part="X1" gate="-2" pin="KL"/>
+<pinref part="RELAY" gate="-2" pin="KL"/>
 <wire x1="-27.94" y1="71.12" x2="-25.4" y2="71.12" width="0.1524" layer="91"/>
 <wire x1="-25.4" y1="71.12" x2="-25.4" y2="48.26" width="0.1524" layer="91"/>
